File: RP2350_V1/RP2350_V1.kicad_sch (KiCad schematic)
At the start: 85 parts, among them J1 Conn_01x04_Pin, J2 Conn_01x08_Socket, J3 USB_C_Receptacle_USB2.0_16P, J4 Conn_01x08_Socket, J5 Conn_01x08_Socket, Q3 Q_PMOS_DGS, SW1 SW_Push_Dual, SW2 SW_Push_Dual, SW3 SW_Push_Dual, SW4 SW_Push_Dual, SW5 SW_Push_Dual, SW6 SW_Push_Dual, SW7 SW_Push_Dual, SW8 SW_Push_Dual, U1 RP2350_60QFN, U2 W25Q128JVS, U3 TPS61200DRC, U4 MCP73812T-420I-OT, U5 NCP1117-3.3_SOT223, U6 74HC14, U7 TPS61202DRC, Y1 ASE-12.000MHZ-ET

Commit message: new power sch, rough lay floorplan
Parts:
- removed BT1: Battery_Cell, symbol Device:Battery_Cell
- removed D1: D_Schottky, symbol Device:D_Schottky
- removed Q3: Q_PMOS_DGS, symbol Device:Q_PMOS_DGS
- removed SW1, SW2, SW3, SW4, SW5, SW6, SW7, SW8: SW_Push_Dual, symbol Switch:SW_Push_Dual
- removed U3: TPS61200DRC, Package_SON:Texas_S-PVSON-N10_ThermalVias, symbol Regulator_Switching:TPS61200DRC
- removed U5: NCP1117-3.3_SOT223, Package_TO_SOT_SMD:SOT-223-3_TabPin2, symbol Regulator_Linear:NCP1117-3.3_SOT223
- removed U7: TPS61202DRC, Package_SON:Texas_S-PVSON-N10_ThermalVias, symbol Regulator_Switching:TPS61202DRC
- added C28: 10p, symbol Device:C
- added C29: 10u, symbol Device:C
- added C30, C31: 22u, symbol Device:C
- added D1: MBR0520LT, Diode_SMD:D_SOD-123, symbol Diode:MBR0520LT
- added IC1, IC2: DMP1045U-7, My_Footprints:SOT96P240X110-3N, symbol My_Library:DMP1045U-7
- added J6: Conn_01x02_Pin, Connector_JST:JST_PH_B2B-PH-K_1x02_P2.00mm_Vertical, symbol Connector:Conn_01x02_Pin
- added R28: 100k, symbol Device:R
- added R29: 1.5Meg, symbol Device:R
- added R30: 1Meg, symbol Device:R
- added R31: 1k, Resistor_SMD:R_0402_1005Metric, symbol Device:R
- added SW1, SW10, SW11, SW12, SW13, SW14, SW4, SW9: PTS 647 SN50 SMTR2 LFS, My_Footprints:PTS 647 SN50 SMTR2 LFS, symbol My_Library:PTS_647_SN50_SMTR2_LFS
- added U3: TPS628110AQWRWYRQ1, My_Footprints:RWY0009A, symbol My_Library:TPS628110AQWRWYRQ1
- added U5: TLV3012AIDBVR, My_Footprints:DBV6, symbol My_Library:TLV3012AIDBVR
- C14: value 1u -> 100n; footprint (none) -> Capacitor_SMD:C_0402_1005Metric
- C15, C21, C22, C23, C24, C25, C26, C27: footprint (none) -> Capacitor_SMD:C_0402_1005Metric
- C16: value 22u -> 100n; footprint (none) -> Capacitor_SMD:C_0402_1005Metric
- C17, C18: footprint (none) -> Capacitor_SMD:C_0805_2012Metric
- C19: value 10u -> 22u
- C2, C3: footprint Capacitor_SMD:C_0805_2012Metric -> Capacitor_SMD:C_0402_1005Metric
- C20: value 10u -> 4.7n; footprint (none) -> Capacitor_SMD:C_0805_2012Metric
- L2: value 2.2u -> 0.47u
- R10: value 2M -> 88.7k
- R11: value 180k -> 19.6k
- R12, R14, R15, R16, R17, R18, R19, R20, R21, R22, R23, R24, R25, R26, R27: footprint (none) -> Resistor_SMD:R_0402_1005Metric
- R13: value 10k -> 100k
- R3: value DNF -> 100k; footprint Resistor_SMD:R_0402_1005Metric -> (none)
- R4: value 0 -> 8.06k; footprint Resistor_SMD:R_0402_1005Metric -> (none)
- R5: value DNF -> 10k
- U2: footprint Package_SO:SOIC-8_5.23x5.23mm_P1.27mm -> My_Footprints:SOIC127P790X216-8N
- U6: footprint (none) -> My_Footprints:SN74HC14DR_D14
Connections:
- net GPIO0 is gone; now on net VBUS: R3.1
- net VAUX is gone; now on net +1V1: C14.1
- net +1V1: now also C15.1, C16.1, U1.23 (DVDD), U1.39 (DVDD), U1.6 (DVDD)
- net +3V3: now also L2.2, R10.1, R13.1, C28.1, C29.1, C30.1, C31.1, R28.1, R29.1, U5.6 (V+); no longer C20.1
- net BTN_BACK: now also U6.2
- net BTN_NEXT: now also U6.6
- net BTN_OK: now also U6.4
- net GND: now also R3.2, R4.2, C29.2, C30.2, C31.2, J6.2 (Pin_2), R28.2, R30.2, SW1.1, SW1.2, SW10.1, SW10.2, SW11.1, SW11.2, SW12.1, SW12.2, SW13.1, SW13.2, SW14.1, SW14.2, SW4.1, SW4.2, SW9.1, SW9.2, U3.4 (GND), U5.2 (V-); no longer R13.2
- net QSPI_SS: now also R5.2, U2.1 (~{CS}); no longer R4.1
- net RUN: now also R31.2
- net VBAT: now also IC1.3 (D), J6.1 (Pin_1)
- net VBUS: now also D1.2 (A), IC1.1 (G), IC2.1 (G); no longer R13.1
- net ~{USB_BOOT}: now also SW4.3, SW4.4
- net at R1.1: now also SW1.3, SW1.4
- net at R16.1, R17.2: now also SW12.3, SW12.4
- net at R20.2, R21.1: now also SW14.3, SW14.4
- net at R22.2, R25.1: now also SW11.3, SW11.4
- net at R18.2, R19.1: now also SW13.3, SW13.4
- net BTN_MACRO_A: now reaches U6.8
- net BTN_MACRO_A: now also U1.3 (GPIO1)
- net at R24.2, R27.1: now also SW10.3, SW10.4
- net BTN_MACRO_C: now reaches U6.12
- net BTN_MACRO_C: now also U1.9 (GPIO6)
- net at R23.2, R26.1: now also SW9.3, SW9.4
- net BTN_MACRO_B: now reaches U6.10
- net BTN_MACRO_B: now also U1.4 (GPIO2)
- removed net FLASH_SS: R3.2, R4.2, R5.2, U2.1 (~{CS})
- net UVLO: no longer names the net of R10.2, R11.1
- net UVLO: now also C28.2, U3.5 (FB)
- removed net V_in: C15.1, L2.1, R10.1
- net V_out_5V: no longer names the net of C19.1
- net V_out_5V: now also D1.1 (K), IC2.3 (D), U3.1 (MODE_SYNC), U3.2 (VIN), U3.8 (EN); no longer C16.1
- new net: R29.2, R30.1, U5.3 (IN+)
- new net: C20.1, U3.6 (SS_TR)
- new net: R31.1, U5.1 (OUT)
- new net: U5.4 (IN-), U5.5 (REF)
- new net: L2.1, U3.3 (SW)
- new net: R4.1, U3.7 (COMP_FSET)
- new net: R13.2, U3.9 (PG)
- new net: IC1.2 (S), IC2.2 (S)
- no-connect marks 9 -> 20
Other:
- note added: "I/O"
- note removed: "Diode prevents boosted battery current from backflowing into the battery and pulling PMOS gate high"
- note removed: "PMOS selects battery power when USB power is disconnected"
- note removed: "Voltage divider sets min output voltage as slightly above 3V (Li-Ion battery considered dead < 3V)"
- note removed: "pull down"
- company: Stefan Praniauskas -> RF Doom
- title: gamer -> VoidLink
- moved on the sheet: C1, C22, H1, H2, H3, H4, R5, U2, U6G

Commit message: First pass routing done! MCU pin updates. UVLO Reset resistor update
Parts:
- removed C12: 10u, Capacitor_SMD:C_0805_2012Metric, symbol Device:C
- removed R28: 100k, symbol Device:R
- added C32: 0.1u, Capacitor_SMD:C_0402_1005Metric, symbol Device:C
- added J7: Conn_01x04_Pin, Connector_PinHeader_2.54mm:PinHeader_1x04_P2.54mm_Vertical, symbol Connector:Conn_01x04_Pin
- C19, C29, C30, C31: footprint (none) -> Capacitor_SMD:C_0805_2012Metric
- C2, C3: footprint Capacitor_SMD:C_0402_1005Metric -> My_Footprints:C_0402_1005Metric_small_pads
- C20: footprint Capacitor_SMD:C_0805_2012Metric -> Capacitor_SMD:C_0402_1005Metric
- C28: footprint (none) -> Capacitor_SMD:C_0402_1005Metric
- J1: footprint Connector_PinSocket_2.54mm:PinSocket_1x04_P2.54mm_Vertical -> Connector_PinHeader_2.54mm:PinHeader_1x04_P2.54mm_Vertical
- L2: footprint (none) -> Inductor_SMD:L_Changjiang_FXL0420
- R10, R11, R13, R29, R3, R30, R4: footprint (none) -> Resistor_SMD:R_0402_1005Metric
- R31: value 1k -> 10k
Connections:
- net +3V3: now also C32.1
- net BTN_BACK: now also U1.7 (GPIO4); no longer U1.5 (GPIO3)
- net BTN_MACRO_A: now also U1.4 (GPIO2); no longer U1.3 (GPIO1)
- net BTN_MACRO_B: now also U1.5 (GPIO3); no longer U1.4 (GPIO2)
- net BTN_MACRO_C: now also U1.10 (GPIO7); no longer U1.9 (GPIO6)
- net BTN_NEXT: now also U1.9 (GPIO6); no longer U1.8 (GPIO5)
- net BTN_OK: now also U1.8 (GPIO5); no longer U1.7 (GPIO4)
- net GND: now also C32.2, J7.2 (Pin_2), J7.4 (Pin_4)
- net SPI0_RX: now also U1.35 (GPIO23); no longer U1.27 (GPIO16)
- net USB_D+: now also D2.2 (K); no longer D2.1 (K)
- net USB_D-: now also D2.1 (K); no longer D2.2 (K)
- net RUN_IN: now reaches R1.1, SW1.3, SW1.4
- net Converter_In: now reaches C19.1, D1.1 (K), IC2.3 (D), U3.1 (MODE_SYNC), U3.2 (VIN), U3.8 (EN)
- net Converter_Out: now reaches L2.1, U3.3 (SW)
- net UART_Tx_DEBUG: now reaches U1.2 (GPIO0)
- net UART_Tx_DEBUG: now also J7.1 (Pin_1)
- new net UART_Rx_DEBUG: J7.3 (Pin_3), U1.3 (GPIO1)
- no-connect marks 20 -> 18
Other:
- moved on the sheet: C22, R1, U6G
