File: RP2350_V1/RP2350_V1.kicad_sch (KiCad schematic)
At the start: 104 parts, among them IC1 DMP1045U-7, IC2 DMP1045U-7, IC3 DMP1045U-7, J1 Conn_01x04_Pin, J2 Conn_01x08_Socket, J3 USB_C_Receptacle_USB2.0_16P, J4 Conn_01x08_Socket, J5 Conn_01x08_Socket, J6 Conn_01x02_Pin, J7 Conn_01x04_Pin, SW1 PTS 647 SN50 SMTR2 LFS, SW10 PTS 647 SN50 SMTR2 LFS, SW11 PTS 647 SN50 SMTR2 LFS, SW12 PTS 647 SN50 SMTR2 LFS, SW13 PTS 647 SN50 SMTR2 LFS, SW14 PTS 647 SN50 SMTR2 LFS, SW4 PTS 647 SN50 SMTR2 LFS, SW9 PTS 647 SN50 SMTR2 LFS, U1 RP2350_60QFN, U2 W25Q128JVS, U3 TPS62811QWRWYRQ1, U4 MCP73812T-420I-OT, U5 TLV3012AIDCKR, U6 74HC14, X1 ABM8-272-T3

Commit message: initial transceier sch
Other:
- added sheet SX1262 (SX1262kicad_sch.kicad_sch)
Changed lines of the file:
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@@
+		)
+	)
+	(sheet
+		(at 85.09 151.13)
+		(size 33.02 53.34)
+		(fields_autoplaced yes)
+		(stroke
+			(width 0.1524)
+			(type solid)
+		)
+		(fill
+			(color 0 0 0 0.0000)
+		)
+		(property "Sheetname" "SX1262"
+			(at 85.09 150.4184 0)
+			(effects
+				(font
+					(size 1.27 1.27)
+				)
+				(justify left bottom)
+			)
+		)
+		(property "Sheetfile" "SX1262kicad_sch.kicad_sch"
+			(at 85.09 205.0546 0)
+			(effects
+				(font
+					(size 1.27 1.27)
+				)
+				(justify left top)
+			)
+		)
+		(instances
+			(project "RP2350_V1"
+				(path "/7f0ba00e-9b42-4d85-a00a-8f4530ab07c8"
+					(page "2")
+				)
+			)
 		)
 	)
