File: RP2350_V1/SX1262kicad_sch.kicad_sch (KiCad schematic)
At the start: 29 parts

Commit message: Transceiver components and schematic final?
Parts:
- U7: LCSC (none) -> C191341
- U8: LCSC (none) -> C470892
Changed lines of the file:
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@@
+			)
+		)
+		(property "LCSC" "C191341"
+			(at 80.01 85.09 0)
+			(effects
+				(font
+					(size 1.27 1.27)
+				)
+				(hide yes)
 			)
 		)
@@
 			(effects
 				(font
+					(size 1.27 1.27)
+				)
+				(hide yes)
+			)
+		)
+		(property "LCSC" "C470892"
+			(at 207.01 73.66 0)
+			(effects
+				(font
