File: RP2350_V2/RP2350_V2-backups/RP2350_V2-2025-03-13_013034/RP2350_V2.kicad_pcb (KiCad board)
At the start: 4 copper layers, 68.8 x 110.6 mm, 140 parts, among them IC1 DMP1045U-7, IC2 DMP1045U-7, IC3 DMP1045U-7, IC4 DMP1045U-7, J1 Conn_01x04_Pin, J3 USB_C_Receptacle_USB2.0_16P, J4 RF_CONNECTOR_5-1814832-2, J5 Conn_01x08_Socket, J6 Conn_01x02_Pin, J7 Conn_01x04_Pin, SW1 PTS 647 SN50 SMTR2 LFS, SW10 PTS 647 SN50 SMTR2 LFS, SW11 PTS 647 SN50 SMTR2 LFS, SW12 PTS 647 SN50 SMTR2 LFS, SW13 PTS 647 SN50 SMTR2 LFS, SW14 PTS 647 SN50 SMTR2 LFS, SW4 PTS 647 SN50 SMTR2 LFS, SW9 PTS 647 SN50 SMTR2 LFS, U1 RP2350_60QFN, U2 W25Q128JVS, U3 TPS62811QWRWYRQ1, U4 MCP73812T-420I-OT, U5 TLV3012AIDCKR, U6 74HC14, X1 ABM8-272-T3

Commit message: optimizations
Parts:
- moved C31 21.3 mm to (151.9, 82.0), turned to 0 degrees
- moved C44 0.63 mm to (143.7, 78.8)
- moved L9 0.60 mm to (144.4, 80.3)
- moved C47 0.40 mm to (146.9, 78.8)
- moved C5 0.36 mm to (140.0, 98.6)
- moved J5 0.35 mm to (135.8, 86.0)
- moved C17 0.35 mm to (135.9, 139.2)
- moved R9 0.24 mm to (145.7, 97.7)
- moved C12 0.24 mm to (145.3, 96.1)
Routing:
- net +3V3: track 182.5 -> 248.5 mm, vias 32 -> 35
- net /SPI1_TX: track 34.4 -> 0.00 mm, vias 2 -> 0
- net /SWCLK: track 37.3 -> 26.7 mm
- net /SWD: track 31.7 -> 23.5 mm
- net /RUN: track 40.0 -> 44.5 mm
- net DIO1: track 33.2 -> 37.6 mm
- net uC_BUSY: track 34.4 -> 38.7 mm
- net GND: track 195.4 -> 191.2 mm, vias 366 -> 365
- net uC_RESET: track 35.3 -> 39.5 mm
- net /SX1262/DIO2: track 25.5 -> 28.5 mm
- net /STATUS_LED: track 26.0 -> 23.6 mm
- net SPIO_RX: track 41.4 -> 43.0 mm
- net Net-(U7-VREG): track 4.16 -> 3.55 mm
